File: Hardware/PQ60-EPS.sch (EAGLE design)
At the start: 32 parts, among them IC1 TPS2552, IC2 TPS2552, IC3 INA3221, X1-BOT FX8C-60S-SV, X1-TOP FX8C-60P-SV

Commit message: Updated to latest PQ60 standard and enhanced circuit,
Parts:
- removed C10, C17, C9: 100nF, rcl:C-EUC0603
- removed CN1: (no value), microbuilder:JST_2PINSH2
- removed IC2: TPS2552, general:TPS2552DBVT
- removed JP1, JP2, JP3, JP4, JP5: (no value), SparkFun-Connectors:M03SMD
- removed R10, R12, R17, R20, R21, R9: 10, rcl:R-EU_R0603
- removed R11, R19, R8: 0R2, rcl:R-EU_R1206
- removed R18, R22: 47k, rcl:R-EU_R0603
- removed SJ1: (no value), SparkFun-Retired:SOLDERJUMPER_2WAYPASTE2&3
- added C3, C5, C6: 100pF, rcl:C-EUC0402
- added C4: 4.7uF 10V, rcl:C-EUC0805
- added C7: 100nF, rcl:C-EUC0603
- added J1: FTS-105-01-L-D, general:FTS-105-01-L-D
- added R1: 10k, rcl:R-EU_R0603
- added TP1: TEST-POINT2, SparkFun-Passives:TEST-POINT2
- added TP2: TEST-POINT3, SparkFun-Passives:TEST-POINT3
- added X2, X3: (no value), SparkFun-Connectors:M04SMD2
- added X4: (no value), SparkFun-Connectors:M03SMD
- added X5: M02SMD, SparkFun-Connectors:M02SMD
- B1: value PQ60-NOPINS -> PQ60-PINS; device general:PQ60-NOPINS -> general:PQ60-PINS; OC_FARNELL (none) -> unknown
- C2: value 100nF -> 100pF; device rcl:C-EUC0603 -> rcl:C-EUC0402; MF (none) -> AVX; MPN (none) -> 02013A101JAT2A; OC_FARNELL unknown -> 2280754
- IC1: value TPS2552 -> LTC4413; device general:TPS2552DBVT -> general:LTC4413EDDPBF; MF (none) -> LINEAR TECHNOLOGY; MPN TPS2552DBVT -> (none); OC_FARNELL 1694421 -> (none); OC_NEWARK 40P3866 -> (none); PACKAGE SOT-23-6 -> (none); SUPPLIER Texas Instruments -> (none)
- IC3: value INA3221 -> MKL05Z32VFM4; device general:INA3221AIRGV -> general:MKL05Z32VFM4; MF TEXAS INSTRUMENTS -> FREESCALE SEMICONDUCTOR; MPN INA3221AIRGVT -> (none); OC_FARNELL 2144251 -> (none)
- IC4: OC_FARNELL (none) -> unknown
- X1-BOT: device PQ60:FX8C-60S-SV -> PQ60:FX8C-60-R2S-SV; OC_FARNELL (none) -> unknown
- X1-TOP: device PQ60:FX8C-60P-SV -> PQ60:FX8C-60-R2P-SV; OC_FARNELL (none) -> unknown
Connections:
- net VIN1 renamed S_ARRAY_1
- net VIN2 renamed S_ARRAY_2
- removed net !3V3_FAULT: IC1./FAULT
- removed net !EN_3V3: IC1.EN
- removed net !EN_VBUS: IC2.EN
- removed net !VBUS_FAULT: IC2./FAULT
- removed net +3V3: C1.1, IC4.VCC, R11.1, R15.2, R16.2, R17.2, X1-BOT.+3.3V@1, X1-BOT.+3.3V@2, X1-BOT.+3.3V@3, X1-TOP.+3.3V@1, X1-TOP.+3.3V@2, X1-TOP.+3.3V@3
- removed net +3V3_OUT: IC1.OUT, R11.2, R12.2
- removed net A0: IC3.A0, SJ1.2
- removed net GPIO[13]: X1-BOT.GPIO13, X1-TOP.GPIO13
- removed net GPIO[14]: X1-BOT.GPIO14, X1-TOP.GPIO14
- removed net ILIMIT_3V3: IC1.ILIM, R18.2
- removed net ILIMIT_VBUS: IC2.ILIM, R22.2
- removed net IN1_N: C10.2, IC3.IN-1, R17.1
- removed net IN1_P: C10.1, IC3.IN+1, R12.1
- removed net IN2_N: C9.2, IC3.IN-2, R10.1
- removed net IN2_P: C9.1, IC3.IN+2, R9.1
- removed net IN3_N: C17.2, IC3.IN-3, R21.1
- removed net IN3_P: C17.1, IC3.IN+3, R20.1
- removed net NC@34: X1-BOT.NC@1, X1-TOP.NC@1
- removed net NC@35: X1-BOT.NC@2, X1-TOP.NC@2
- removed net NC@36: X1-BOT.NC@3, X1-TOP.NC@3
- removed net NC@42: X1-BOT.NC@5, X1-TOP.NC@5
- removed net NC@43: X1-BOT.NC@6, X1-TOP.NC@6
- removed net NC@56: X1-BOT.NC@7, X1-TOP.NC@7
- removed net POWER_CRIT: IC3.CRIT
- removed net POWER_SEQ: IC3.TC
- removed net POWER_VALID: IC3.PV
- removed net POWER_WARN: IC3.WARN
- removed net SOLAR_1: JP1.3
- removed net SOLAR_2: JP2.3
- removed net SOLAR_3: JP3.3
- removed net SOLAR_4: JP4.3
- removed net SPI_CS: X1-BOT.SS, X1-TOP.SS
- removed net STAT1: IC1.STAT
- removed net STAT2: IC2.STAT
- removed net TA1: JP1.2
- removed net TA2: JP2.2
- removed net TA3: JP3.2
- removed net TA4: JP4.2
- removed net USB_N: X1-BOT.USB_N, X1-TOP.USB_N
- removed net USB_P: X1-BOT.USB_P, X1-TOP.USB_P
- removed net VBUS: R10.2, R8.1, X1-BOT.VBUS@1, X1-BOT.VBUS@2, X1-BOT.VBUS@3, X1-TOP.VBUS@1, X1-TOP.VBUS@2, X1-TOP.VBUS@3
- removed net VBUS_OUT: IC2.OUT, R8.2, R9.2
- removed net VBUS_SW[1]: X1-BOT.VBUS_SW1, X1-TOP.VBUS_SW1
- removed net VBUS_SW[2]: X1-BOT.VBUS_SW2, X1-TOP.VBUS_SW2
- removed net VBUS_SW[3]: X1-BOT.VBUS_SW3, X1-TOP.VBUS_SW3
- removed net VIN3: IC2.INA
- removed net VIN4: IC2.INB
- removed net VSOL_SEN: R19.1, R21.2
- removed net ~SHDN: IC1.~SHDN
- new net !SHDN!: IC1.!SHDN!
- new net +3V3_I_SEN: IC3.PTB2/IRQ_10/LLWU_P5
- new net +3V3_SW[0]_!FAULT!: IC3.PTB11
- new net +3V3_SW[1]_!FAULT!: IC3.PTB10
- new net +3V3_SW[1]_EN: IC3.PTB9
- new net +3V3_SW[2]_!FAULT!: IC3.PTB8
- new net +3V3_SW[2]_EN: IC3.PTA6/LLWU_P2
- new net +3V3_SW[3]_!FAULT!: IC3.PTA5/LLWU_P1/RTC_CLK_IN
- new net +3V3_SW[3]_EN: IC3.PTA4/LLWU_P0
- new net +3V3_V_SEN: IC3.PTA8
- new net BMS_!CHG!: IC3.PTA10/IRQ_12
- new net BMS_!PGD!: IC3.PTA9
- new net GPIO[0]: X1-BOT.GPIO0@25, X1-TOP.GPIO0@25
- new net I2C_INT: IC3.PTB5/IRQ_16, TP2.1
- new net IDIODE_STAT: IC1.STAT, IC3.PTA11/IRQ_13
- new net IN_SEN: IC1.EN, IC1.IN, IC3.IN, IC4.IN
- new net I_LIM_SW2: IC3.ILIM
- new net I_LIM_SW3: IC4.ILIM
- new net I_LIM_VCC: IC1.ILIM, R1.1
- new net MPPT_PGD: IC3.PTA12/IRQ_17/LPTMR0_ALT2
- new net N$3: B1.3, C5.1
- new net N$4: B1.4, C6.1
- new net N$5: IC3.VREFH, TP1.1
- new net OUT: IC1.OUT
- new net OUT_!FAULT!: IC1.~FAULT
- new net OUT_SW2: IC3.OUT
- new net OUT_SW3: IC4.OUT
- new net PRO1: C1.1, IC4.VCC, R15.2, R16.2, X1-BOT.+3V3@57, X1-BOT.+3V3@58, X1-BOT.+3V3@59, X1-BOT.+3V3@60, X1-TOP.+3V3@57, X1-TOP.+3V3@58, X1-TOP.+3V3@59, X1-TOP.+3V3@60
- new net RESET: IC3.PTA1/IRQ_1/LPTMR0_ALT1, J1.!RESET, R1.1
- new net SOLAR[1..2]: X2.2, X2.4
- new net SOLAR[3..4]: X3.2, X3.4
- new net SW2_!FAULT!: IC3.~FAULT
- new net SW2_EN: IC3.EN
- new net SW3_!FAULT!: IC4.~FAULT
- new net SW3_EN: IC4.EN
- new net SWD_CLK: IC3.PTA0/IRQ_0/LLWU_P7, J1.SWDCLK/TCK
- new net SWD_DIO: IC3.PTA2, J1.SWDIO/TMS
- new net VBAT_I_SEN: IC3.PTB0/IRQ_8/LLWU_P4
- new net VBAT_SW[0]_!FAULT!: IC3.PTA7/IRQ_7/LLWU_P3
- new net VBAT_SW[1]: X1-BOT.VBAT_SW1@13, X1-BOT.VBAT_SW1@14, X1-TOP.VBAT_SW1@13, X1-TOP.VBAT_SW1@14
- new net VBAT_SW[1]_!FAULT!: IC3.PTA13
- new net VBAT_SW[1]_EN: IC3.PTA3
- new net VBAT_SW[2]: X1-BOT.VBAT_SW2@17, X1-BOT.VBAT_SW2@18, X1-TOP.VBAT_SW2@17, X1-TOP.VBAT_SW2@18
- new net VBAT_SW[2]_!FAULT!: IC3.PTB12
- new net VBAT_SW[2]_EN: IC3.PTB7/IRQ_3
- new net VBAT_SW[3]: X1-BOT.VBAT_SW3@21, X1-BOT.VBAT_SW3@22, X1-TOP.VBAT_SW3@21, X1-TOP.VBAT_SW3@22
- new net VBAT_SW[3]_!FAULT!: IC3.PTB13
- new net VBAT_SW[3]_EN: IC3.PTB6/IRQ_2/LPTMR0_ALT3
- new net VBAT_V_SEN: IC3.PTB1/IRQ_9
- new net V_BAT: X4.3
- net !RST: now also X1-BOT./RST@27, X1-TOP./RST@27; no longer X1-BOT.RST, X1-TOP.RST
- net +3V3_SW[1]: now also X1-BOT.+3V3_SW1@1, X1-BOT.+3V3_SW1@2, X1-TOP.+3V3_SW1@1, X1-TOP.+3V3_SW1@2; no longer X1-BOT.+3.3V_SW1, X1-TOP.+3.3V_SW1
- net +3V3_SW[2]: now also X1-BOT.+3V3_SW2@5, X1-BOT.+3V3_SW2@6, X1-TOP.+3V3_SW2@5, X1-TOP.+3V3_SW2@6; no longer X1-BOT.+3.3V_SW2, X1-TOP.+3.3V_SW2
- net +3V3_SW[3]: now also X1-BOT.+3.3V_SW3@10, X1-BOT.+3.3V_SW3@9, X1-TOP.+3.3V_SW3@10, X1-TOP.+3.3V_SW3@9; no longer X1-BOT.+3.3V_SW3, X1-TOP.+3.3V_SW3
- net +3V3_UNPRO: now also C7.1, IC3.VDD, J1.VCC, R1.2; no longer IC1.IN
- net BATT_PROG: now also R1.2
- net GND: now also C3.2, C4.1, C4.2, C5.2, C6.2, C7.2, IC1.GND@6, IC1.GND@7, IC3.THERMAL_PAD, IC3.VREFL, IC3.VSS, IC4.EP, J1.GND@3, J1.GND@5, J1.GND_DET, J1.KEY, R1.1, R1.2, X1-BOT.GND@28, X1-BOT.RTN_3V3@53, X1-BOT.RTN_3V3@54, X1-BOT.RTN_3V3@55, X1-BOT.RTN_3V3@56, X1-BOT.RTN_3V3_SW1@3, X1-BOT.RTN_3V3_SW1@4, X1-BOT.RTN_3V3_SW2@7, X1-BOT.RTN_3V3_SW2@8, X1-BOT.RTN_3V3_SW3@11, X1-BOT.RTN_3V3_SW3@12, X1-BOT.RTN_VBAT@45, X1-BOT.RTN_VBAT@46, X1-BOT.RTN_VBAT@47, X1-BOT.RTN_VBAT@48, X1-BOT.RTN_VBAT_SW1@15, X1-BOT.RTN_VBAT_SW1@16, X1-BOT.RTN_VBAT_SW2@19, X1-BOT.RTN_VBAT_SW2@20, X1-BOT.RTN_VBAT_SW3@23, X1-BOT.RTN_VBAT_SW3@24, X1-TOP.GND@28, X1-TOP.RTN_3V3@53, X1-TOP.RTN_3V3@54, X1-TOP.RTN_3V3@55, X1-TOP.RTN_3V3@56, X1-TOP.RTN_3V3_SW1@3, X1-TOP.RTN_3V3_SW1@4, X1-TOP.RTN_3V3_SW2@7, X1-TOP.RTN_3V3_SW2@8, X1-TOP.RTN_3V3_SW3@11, X1-TOP.RTN_3V3_SW3@12, X1-TOP.RTN_VBAT@45, X1-TOP.RTN_VBAT@46, X1-TOP.RTN_VBAT@47, X1-TOP.RTN_VBAT@48, X1-TOP.RTN_VBAT_SW1@15, X1-TOP.RTN_VBAT_SW1@16, X1-TOP.RTN_VBAT_SW2@19, X1-TOP.RTN_VBAT_SW2@20, X1-TOP.RTN_VBAT_SW3@23, X1-TOP.RTN_VBAT_SW3@24, X2.1, X2.3, X3.1, X3.3, X4.1; no longer IC1.GND@1, IC1.GND@2, IC2.ENBA, IC2.ENBB, IC2.EP, IC2.GND, JP1.1, JP2.1, JP3.1, JP4.1, JP5.1, R18.1, R22.1, SJ1.3, X1-BOT.GND@1, X1-BOT.GND@10, X1-BOT.GND@11, X1-BOT.GND@12, X1-BOT.GND@13, X1-BOT.GND@14, X1-BOT.GND@15, X1-BOT.GND@16, X1-BOT.GND@17, X1-BOT.GND@18, X1-BOT.GND@19, X1-BOT.GND@2, X1-BOT.GND@3, X1-BOT.GND@4, X1-BOT.GND@5, X1-BOT.GND@6, X1-BOT.GND@7, X1-BOT.GND@8, X1-BOT.GND@9, X1-TOP.GND@1, X1-TOP.GND@10, X1-TOP.GND@11, X1-TOP.GND@12, X1-TOP.GND@13, X1-TOP.GND@14, X1-TOP.GND@15, X1-TOP.GND@16, X1-TOP.GND@17, X1-TOP.GND@18, X1-TOP.GND@19, X1-TOP.GND@2, X1-TOP.GND@3, X1-TOP.GND@4, X1-TOP.GND@5, X1-TOP.GND@6, X1-TOP.GND@7, X1-TOP.GND@8, X1-TOP.GND@9
- net GPIO[10]: now also X1-BOT.GPIO10@42, X1-TOP.GPIO10@42; no longer X1-BOT.GPIO10, X1-TOP.GPIO10
- net GPIO[11]: now also X1-BOT.GPIO11@43, X1-TOP.GPIO11@43; no longer X1-BOT.GPIO11, X1-TOP.GPIO11
- net GPIO[12]: now also X1-BOT.GPIO12@44, X1-TOP.GPIO12@44; no longer X1-BOT.GPIO12, X1-TOP.GPIO12
- net GPIO[1]: now also X1-BOT.GPIO1@26, X1-TOP.GPIO1@26; no longer X1-BOT.GPIO1, X1-TOP.GPIO1
- net GPIO[2]: now also X1-BOT./SS/GPIO2@34, X1-TOP./SS/GPIO2@34; no longer X1-BOT.GPIO2, X1-TOP.GPIO2
- net GPIO[3]: now also X1-BOT.GPIO3@35, X1-TOP.GPIO3@35; no longer X1-BOT.GPIO3, X1-TOP.GPIO3
- net GPIO[4]: now also X1-BOT.GPIO4@36, X1-TOP.GPIO4@36; no longer X1-BOT.GPIO4, X1-TOP.GPIO4
- net GPIO[5]: now also X1-BOT.GPIO5@37, X1-TOP.GPIO5@37; no longer X1-BOT.GPIO5, X1-TOP.GPIO5
- net GPIO[6]: now also X1-BOT.GPIO6@38, X1-TOP.GPIO6@38; no longer X1-BOT.GPIO6, X1-TOP.GPIO6
- net GPIO[7]: now also X1-BOT.GPIO7@39, X1-TOP.GPIO7@39; no longer X1-BOT.GPIO7, X1-TOP.GPIO7
- net GPIO[8]: now also X1-BOT.GPIO8@40, X1-TOP.GPIO8@40; no longer X1-BOT.GPIO8, X1-TOP.GPIO8
- net GPIO[9]: now also X1-BOT.GPIO9@41, X1-TOP.GPIO9@41; no longer X1-BOT.GPIO9, X1-TOP.GPIO9
- net I2C_SCL: now also IC3.PTB3/IRQ_14, X1-BOT.SCL@29, X1-TOP.SCL@29; no longer IC3.SCL, X1-BOT.SCL, X1-TOP.SCL
- net I2C_SDA: now also IC3.PTB4/IRQ_15/LLWU_P6, X1-BOT.SDA@30, X1-TOP.SDA@30; no longer IC3.SDA, X1-BOT.SDA, X1-TOP.SDA
- net LDO: now also C4.2
- net MPPC: now also R1.2
- net N$1: now also B1.1, C2.1
- net N$2: now also B1.2, C3.1
- net SPI_MISO: now also X1-BOT.MISO@32, X1-TOP.MISO@32; no longer X1-BOT.MISO, X1-TOP.MISO
- net SPI_MOSI: now also X1-BOT.MOSI@31, X1-TOP.MOSI@31; no longer X1-BOT.MOSI, X1-TOP.MOSI
- net SPI_SCK: now also X1-BOT.SCK@33, X1-TOP.SCK@33; no longer X1-BOT.SCK, X1-TOP.SCK
- net THM: now also C5.1, R1.1, X4.2; no longer JP5.2
- net VBAT: now also X1-BOT.VBAT@49, X1-BOT.VBAT@50, X1-BOT.VBAT@51, X1-BOT.VBAT@52, X1-TOP.VBAT@49, X1-TOP.VBAT@50, X1-TOP.VBAT@51, X1-TOP.VBAT@52; no longer JP5.3
- net VOUT: now also C3.1; no longer IC1.OUTA, IC1.OUTB, IC2.OUTA, IC2.OUTB
- net VSOL: now also C4.1, IC1.OUTA, IC1.OUTB; no longer R19.2, R20.2
- net VSYS: now also X5.2; no longer CN1.1
- net VSYS_SW: now also X5.1; no longer C2.1, CN1.2, IC2.IN, IC3.VPU, IC3.VS, SJ1.1
Other:
- note added: "1V = 4A"
- note added: "1V = 5.1V"
- note added: "2 analogue outs (1V max) 4 digital outs 3 digital ins"
- note added: "Replace with TPS630250"
- note added: "sw: I2C/SMBus/PMBus interface 2 output blocks MPPT Status IDiode Status BMS Status SMPS Status"
- note removed: "Ilimit = 23950Volts / Rlimit"
- note removed: "de-coupling cap"
- moved on the sheet: C2, R15, R16
